File: 15_XCAN.sch (KiCad schematic (older format))
At the start: 16 parts, among them J1 Conn_01x01, J2 Conn_01x01, J3 Conn_01x01, J4 Conn_01x01, J5 Conn_01x01, J6 Conn_01x01, J7 Conn_01x01, U1 MCP2551-I-SN

Commit message: maj split librairies
Parts:
- H1, H2, H3, H4, H5, H6: footprint Chimere:trou -> Chimere_comps:trou
- J1, J2, J3, J4, J5, J6, J7: footprint Chimere:Castellated_conn -> Chimere_mods:Castellated_conn
Changed lines of the file:
@@
 F 0 "J1" H 4255 1317 50  0000 L CNN
 F 1 "Conn_01x01" H 4255 1226 50  0000 L CNN
-F 2 "Chimere:Castellated_conn" H 4175 1275 50  0001 C CNN
+F 2 "Chimere_mods:Castellated_conn" H 4175 1275 50  0001 C CNN
 F 3 "~" H 4175 1275 50  0001 C CNN
 	1    4175 1275
@@
 F 0 "J3" H 4255 1667 50  0000 L CNN
 F 1 "Conn_01x01" H 4255 1576 50  0000 L CNN
-F 2 "Chimere:Castellated_conn" H 4175 1625 50  0001 C CNN
+F 2 "Chimere_mods:Castellated_conn" H 4175 1625 50  0001 C CNN
 F 3 "~" H 4175 1625 50  0001 C CNN
 	1    4175 1625
@@
 F 0 "J2" H 4255 1492 50  0000 L CNN
 F 1 "Conn_01x01" H 4255 1401 50  0000 L CNN
-F 2 "Chimere:Castellated_conn" H 4175 1450 50  0001 C CNN
+F 2 "Chimere_mods:Castellated_conn" H 4175 1450 50  0001 C CNN
 F 3 "~" H 4175 1450 50  0001 C CNN
 	1    4175 1450
@@
 F 0 "J5" H 4255 2017 50  0000 L CNN
 F 1 "Conn_01x01" H 4255 1926 50  0000 L CNN
-F 2 "Chimere:Castellated_conn" H 4175 1975 50  0001 C CNN
+F 2 "Chimere_mods:Castellated_conn" H 4175 1975 50  0001 C CNN
 F 3 "~" H 4175 1975 50  0001 C CNN
 	1    4175 1975
@@
 F 0 "J4" H 4255 1842 50  0000 L CNN
 F 1 "Conn_01x01" H 4255 1751 50  0000 L CNN
-F 2 "Chimere:Castellated_conn" H 4175 1800 50  0001 C CNN
+F 2 "Chimere_mods:Castellated_conn" H 4175 1800 50  0001 C CNN
 F 3 "~" H 4175 1800 50  0001 C CNN
 	1    4175 1800
@@
 F 0 "H1" H 4575 6996 50  0000 L CNN
 F 1 "percage" H 4575 6905 50  0000 L CNN
-F 2 "Chimere:trou" H 4475 6950 50  0001 C CNN
+F 2 "Chimere_comps:trou" H 4475 6950 50  0001 C CNN
 F 3 "~" H 4475 6950 50  0001 C CNN
 	1    4475 6950
@@
 F 0 "H5" H 4575 7271 50  0000 L CNN
 F 1 "percage" H 4575 7180 50  0000 L CNN
-F 2 "Chimere:trou" H 4475 7225 50  0001 C CNN
+F 2 "Chimere_comps:trou" H 4475 7225 50  0001 C CNN
 F 3 "~" H 4475 7225 50  0001 C CNN
 	1    4475 7225
@@
 F 0 "H2" H 5125 6996 50  0000 L CNN
 F 1 "percage" H 5125 6905 50  0000 L CNN
-F 2 "Chimere:trou" H 5025 6950 50  0001 C CNN
+F 2 "Chimere_comps:trou" H 5025 6950 50  0001 C CNN
 F 3 "~" H 5025 6950 50  0001 C CNN
 	1    5025 6950
@@
 F 0 "H6" H 5125 7271 50  0000 L CNN
 F 1 "percage" H 5125 7180 50  0000 L CNN
-F 2 "Chimere:trou" H 5025 7225 50  0001 C CNN
+F 2 "Chimere_comps:trou" H 5025 7225 50  0001 C CNN
 F 3 "~" H 5025 7225 50  0001 C CNN
 	1    5025 7225
@@
 F 0 "H3" H 5600 6996 50  0000 L CNN
 F 1 "percage" H 5600 6905 50  0000 L CNN
-F 2 "Chimere:trou" H 5500 6950 50  0001 C CNN
+F 2 "Chimere_comps:trou" H 5500 6950 50  0001 C CNN
 F 3 "~" H 5500 6950 50  0001 C CNN
 	1    5500 6950
@@
 F 0 "H4" H 6150 6996 50  0000 L CNN
 F 1 "percage" H 6150 6905 50  0000 L CNN
-F 2 "Chimere:trou" H 6050 6950 50  0001 C CNN
+F 2 "Chimere_comps:trou" H 6050 6950 50  0001 C CNN
 F 3 "~" H 6050 6950 50  0001 C CNN
 	1    6050 6950
@@
 F 0 "J6" H 4255 2192 50  0000 L CNN
 F 1 "Conn_01x01" H 4255 2101 50  0000 L CNN
-F 2 "Chimere:Castellated_conn" H 4175 2150 50  0001 C CNN
+F 2 "Chimere_mods:Castellated_conn" H 4175 2150 50  0001 C CNN
 F 3 "~" H 4175 2150 50  0001 C CNN
 	1    4175 2150
@@
 F 0 "J7" H 5605 1342 50  0000 L CNN
 F 1 "Conn_01x01" H 5605 1251 50  0000 L CNN
-F 2 "Chimere:Castellated_conn" H 5525 1300 50  0001 C CNN
+F 2 "Chimere_mods:Castellated_conn" H 5525 1300 50  0001 C CNN
 F 3 "~" H 5525 1300 50  0001 C CNN
 	1    5525 1300
