File: 15_XCAN.kicad_pcb (KiCad board)
At the start: 2 copper layers, 20.3 x 20.3 mm, 16 parts, among them J1 Conn_01x01, J2 Conn_01x01, J3 Conn_01x01, J4 Conn_01x01, J5 Conn_01x01, J6 Conn_01x01, J7 Conn_01x01, U1 MCP2551-I-SN

Commit message: maj split librairies
Parts:
- H1, H2, H3, H4, H5, H6: footprint Chimere:trou -> Chimere_comps:trou
- J1, J2, J3, J4, J5, J6, J7: footprint Chimere:Castellated_conn -> Chimere_mods:Castellated_conn

Commit message: maj kicad v6
Other:
- net class Default removed
- net class demi-gros removed
- net class gros removed
